File: eagle/808_cowbell.sch (EAGLE design)
At the start: 72 parts, among them Q1* 2SC945, Q14* 2SC945, Q15* 2SC945, Q35 2SC828, Q5* 2SA733, U1 4584N, U2 µPC4558C, U24 µPC4558C, U6 µPC4558C

Commit message: routed and cammed
Parts:
- removed C28*: 10n, TR808clone:C-EU3.5MM_PITCH
- removed C29: 47/16, TR808clone:CPOL-EUE2.5-5
- removed C29*: 3.3n, TR808clone:C-EU3.5MM_PITCH
- removed C30*, C31*: 2.2n, TR808clone:C-EU3.5MM_PITCH
- removed C31, C34*, C75*: 1/50, TR808clone:CPOL-EUE2.5-5
- removed C32: 39n, TR808clone:C-EU050-024X044
- removed C32*, C33*: 10/16, TR808clone:CPOL-EUE2.5-5
- removed C33, C5*: 18n, TR808clone:C-EU4MM_PITCH
- removed C6*, C76*: 22n, TR808clone:C-EU4MM_PITCH
- removed C9*: .47/50, TR808clone:CPOL-EUE2.5-5
- removed D1*, D2*, D3*, D4*: 1N4148DO35-7, TR808clone:1N4148DO35-7
- removed Q1*, Q14*, Q15*: 2SC945, TR808clone:2SC945
- removed Q35: 2SC828, 808:2SC828
- removed Q5*: 2SA733, TR808clone:2SA733
- removed R116*: 8K2, TR808clone:R-EU_0207/5V
- removed R117*, R132, R133, R4*, R9*: 22K, TR808clone:R-EU_0207/5V
- removed R122*, R163*: 1K, TR808clone:R-EU_0207/5V
- removed R124, R31*, R33*: 100R, TR808clone:R-EU_0207/5V
- removed R127: 47K, TR808clone:R-EU_0207/5V
- removed R128, R130: 1M, TR808clone:R-EU_0207/5V
- removed R129: 330K, TR808clone:R-EU_0207/5V
- removed R131: 300K, TR808clone:R-EU_0207/5V
- removed R14*: 4K7, TR808clone:R-EU_0207/5V
- removed R18*, R21*, R22*: 3K3, TR808clone:R-EU_0207/5V
- removed R19*, R28*, R29*, R45*: 100K, TR808clone:R-EU_0207/5V
- removed R20*: 15K, TR808clone:R-EU_0207/5V
- removed R23*: 100K, TR808clone:R-EU_0207/2V
- removed R24*, R63*, R65*: 2K2, TR808clone:R-EU_0207/5V
- removed R25*, R30*, R32*: 470K, TR808clone:R-EU_0207/5V
- removed R26*, R5*: 10K, TR808clone:R-EU_0207/5V
- removed R27*: 10K, TR808clone:R-EU_0207/2V
- removed R44*: 150K, TR808clone:R-EU_0207/5V
- removed R62*, R64*, R82*: 33K, TR808clone:R-EU_0207/5V
- removed TM1*, TM2*: 220KB, TR808clone:TRIM_EU-CT6
- removed TM4: 22KB, TR808clone:TRIM_EU-CT6
- removed U2, U24, U6: µPC4558C, TR808clone:µPC4558C
- removed VR5*: 5KA, TR808clone:POT_808
- added 540HZ, 800HZ: 200k, pot:3RP/1610N
- added ACCENT, OUTPUT, TRIGGER: LSP11, solpad:LSP11
- added C1, C14: 22n, TR808clone:C-EU4MM_PITCH
- added C10: 3.3n, TR808clone:C-EU3.5MM_PITCH
- added C11: 10n, TR808clone:C-EU3.5MM_PITCH
- added C12: 0.1uF, TR808clone:C-EU3.5MM_PITCH
- added C13, C9: 1/50, TR808clone:CPOL-EUE2.5-5
- added C15: .47/50, TR808clone:CPOL-EUE2.5-5
- added C2: 18n, TR808clone:C-EU4MM_PITCH
- added C3, C4: 10/16, TR808clone:CPOL-EUE2.5-5
- added C5, C6: 22p, TR808clone:C-EU025-025X050
- added C7, C8: 2.2n, TR808clone:C-EU3.5MM_PITCH
- added D1, D2, D3, D4: 1N4148DO35-7, TR808clone:1N4148DO35-7
- added IC1: 4584N, TR808clone:4584N
- added IC2: TL072P, linear:TL072P
- added LEVEL: 5KA, pot:3RP/1610N
- added R1, R2: 20K, TR808clone:R-EU_0207/5V
- added R10, R20, R9: 2K2, TR808clone:R-EU_0207/5V
- added R11, R12, R21: 470K, TR808clone:R-EU_0207/5V
- added R13, R14: 100R, TR808clone:R-EU_0207/5V
- added R15, R16, R5: 100K, TR808clone:R-EU_0207/5V
- added R17: 10K, TR808clone:R-EU_0207/7
- added R18, R26: 10K, TR808clone:R-EU_0207/5V
- added R19, R7, R8: 33K, TR808clone:R-EU_0207/5V
- added R22, R25, R28, R29: 22K, TR808clone:R-EU_0207/5V
- added R23: 8K2, TR808clone:R-EU_0207/5V
- added R27: 4K7, TR808clone:R-EU_0207/5V
- added R30, R31: 1K, TR808clone:R-EU_0207/5V
- added R6: 150K, TR808clone:R-EU_0207/5V
- added T1, T2, T3: BC639, transistor:BC639-NPN-TO92-ECB
- added T4: BC640, transistor:BC640-PNP-TO92-BCE
- U1: value 4584N -> POWER; device TR808clone:4584N -> eurorack:POWER
Connections:
- removed net +B1*: R30*.2, R32*.2, U2G$3.V+
- removed net +B5: R124.2, U24G$3.V+
- removed net -B1*: U2G$3.V-
- removed net -B5: U24G$3.V-
- removed net CB: R4*.2
- removed net N$179: D1*.A, R18*.1, R20*.2
- removed net N$187: C5*.2, TM2*.E, U1E.I
- removed net N$189: C6*.2, TM1*.E, U1F.I
- removed net N$213: R45*.1, TM2*.S
- removed net N$214: R44*.1, TM1*.S
- removed net N$222: R19*.1, R20*.1, R21*.2, U2A.+IN
- removed net N$224: R22*.2, R23*.1, U2A.-IN
- removed net N$228: R127.2, TM4.A
- removed net N$280: C31.-, R131.1, U24A.+IN
- removed net N$489: R129.1, R130.2, TM4.S
- removed net N$490: R129.2, U24A.-IN
- removed net N$491: C31.+, Q35.E, R128.1
- removed net N$492: C29.+, R124.1, R128.2
- removed net N$493: C32.1, R132.1, R133.2
- removed net N$494: C33.1, R132.2, U24B.+IN
- removed net PN: C32.2, U24B.-IN, U24B.OUT
- removed net TP6: R44*.2, R62*.1, U1F.O
- removed net TRIG: R18*.2, R19*.2
- removed net WN: R130.1, R133.1, U24A.OUT
- new net +12V: C5.2, IC2P.V+, R11.2, R12.2, U1.+12V
- new net +5V: IC1A.I, IC1B.I, IC1C.I, IC1D.I, IC1P.VDD, U1.+5V
- new net -12V: C6.2, IC2P.V-, U1.-12V
- new net N$1: C2.2, IC1E.I, R2.1
- new net N$2: C1.2, IC1F.I, R1.1
- new net N$24: C12.1, D3.C, R22.2
- new net N$25: C12.2, R25.2
- new net N$26: D3.A, TRIGGER.MP
- new net N$3: 800HZ.S, R5.1
- new net N$4: 540HZ.S, R6.1
- new net N$5: IC1F.O, R6.2, R7.1
- new net N$6: 540HZ.E, R1.2
- new net N$7: 800HZ.E, R2.2
- net CB_OUT: now also OUTPUT.MP, R31.2; no longer R163*.2
- net GND: now also C1.1, C15.-, C2.1, C5.1, C6.1, C9.-, IC1P.VSS, IC2A.+IN, LEVEL.A, R10.2, R13.1, R14.1, R20.1, R22.1, R26.1, R29.2, R9.2, T3.E, U1.GND; no longer C29.-, C33.2, C34*.-, C5*.1, C6*.1, C9*.-, D1*.C, Q1*.E, Q35.B, R117*.2, R127.1, R131.2, R21*.1, R22*.1, R24*.1, R31*.1, R33*.1, R5*.1, R63*.2, R65*.2, U1P.VSS, U2B.+IN, VR5*G$1.A, VR5*G$2.C
- net N$441: now also R27.1, R28.2, T4.B; no longer Q5*.B, R14*.1, R9*.2
- net N$442: now also R28.1, T3.C; no longer Q1*.C, R9*.1
- net N$443: now also R25.1, R26.2, T3.B; no longer Q1*.B, R4*.1, R5*.2
- net N$444: now also C15.+, D4.C, R15.2, R16.2, R19.1; no longer C9*.+, D2*.C, R28*.2, R29*.2, R82*.1
- net N$445: now also R13.2, T1.E; no longer Q15*.E, R31*.2
- net N$446: now also C3.+, R11.1, T1.B; no longer C32*.+, Q15*.B, R30*.1
- net N$447: now also D1.C, T1.C; no longer D3*.C, Q15*.C
- net N$448: now also D1.A, R15.1, R18.2; no longer D3*.A, R26*.2, R28*.1
- net N$449: now also R14.2, T2.E; no longer Q14*.E, R33*.2
- net N$450: now also C4.+, R12.1, T2.B; no longer C33*.+, Q14*.B, R32*.1
- net N$451: now also D2.C, T2.C; no longer D4*.C, Q14*.C
- net N$452: now also D2.A, R16.1, R17.2; no longer D4*.A, R27*.2, R29*.1
- net N$453: now also C8.1, R18.1; no longer C30*.1, R26*.1
- net N$454: now also C7.1, R17.1; no longer C31*.1, R27*.1
- net N$455: now also C10.1, C11.1, C7.2, C8.2, R20.2; no longer C28*.1, C29*.1, C30*.2, C31*.2, R24*.2
- net N$456: now also C10.2, C13.-, IC2A.OUT, R21.1; no longer C29*.2, C75*.-, R25*.1, U2B.OUT
- net N$457: now also C11.2, IC2A.-IN, R21.2; no longer C28*.2, R25*.2, U2B.-IN
- net N$458: now also IC2B.-IN, IC2B.OUT, R31.1; no longer R163*.1, U6A.-IN, U6A.OUT
- net N$459: now also C14.2, IC2B.+IN, R29.1; no longer C76*.2, R117*.1, U6A.+IN
- net N$460: now also C14.1, LEVEL.S; no longer C76*.1, VR5*G$1.S
- net N$461: now also LEVEL.E, R23.2; no longer R116*.2, VR5*G$1.E
- net N$462: now also C13.+, R23.1; no longer C75*.+, R116*.1
- net N$464: now also C3.-, R7.2, R9.1; no longer C32*.-, R62*.2, R63*.1
- net N$465: now also C4.-, R10.1, R8.2; no longer C33*.-, R64*.2, R65*.1
- net N$466: now also C9.+, R19.2; no longer C34*.+, R82*.2
- net N$467: now also R30.2, T4.C; no longer Q5*.C, R122*.2
- net N$468: now also D4.A, R30.1; no longer D2*.A, R122*.1
- net TP7: now also IC1E.O, R5.2, R8.1; no longer R45*.2, R64*.1, U1E.O
- net TRIG*: now also ACCENT.MP, R27.2, T4.E; no longer Q5*.E, R14*.2, R23*.2, U2A.OUT
Other:
- note removed: "Noise"
